File: IEEE_Wrkshp_08192026.kicad_sch (KiCad schematic)
At the start: 0 parts

Commit message: Schematic - Added Rectifier Circuit and need to do Analysis
Parts:
- added C1: 470u, symbol Device:C_Polarized_US
- added C2: C, symbol Device:C
- added D1, D2, D3, D4: D_45deg, symbol Device:D_45deg
- added D5: D_Zener, symbol Device:D_Zener
- added D6: LED, symbol Device:LED
- added J1: Screw_Terminal_01x02, symbol Connector:Screw_Terminal_01x02
- added J2: Screw_Terminal_01x03, symbol Connector:Screw_Terminal_01x03
- added Q1: RS9N50D, Package_TO_SOT_SMD:TO-252-2, symbol Transistor_FET:RS9N50D
- added R1, R2, R5, R6, R7: R_US, symbol Device:R_US
- added R3, R4: R, symbol Device:R_Small_US
- added T1: Transformer_1P_1S, symbol Device:Transformer_1P_1S
- added U1: Opamp_Dual, symbol Device:Opamp_Dual
Connections:
- new net: C2.1, D6.2 (A), J1.1 (Pin_1), Q1.3 (S), R5.1
- new net: Q1.1 (G), U1.1
- new net: D6.1 (K), R7.1
- new net: R3.2, R4.1, U1.3 (+)
- new net AC_Pin1: J2.1 (Pin_1), T1.1 (AA)
- new net AC_Pin2: J2.2 (Pin_2), T1.2 (AB)
- new net AC_Rectified_V+: C1.1, D3.1 (K), D4.1 (K), D5.1 (K), Q1.2 (D), R1.1, R3.1, U1.8 (V+)
- new net AC_Rectified_V-: C1.2, D1.2 (A), D2.2 (A), D5.2 (A), R2.2, U1.4 (V-)
- new net Earth: J2.3 (Pin_3)
- new net T1: D1.1 (K), D3.2 (A), T1.4 (SB)
- new net T2: D2.1 (K), D4.2 (A), T1.3 (SA)
- new net VirtualGND: C2.2, J1.2 (Pin_2), R1.2, R2.1, R4.2, R6.2, R7.2
- new net Vref: R5.2, R6.1, U1.2 (-)
- no-connect marks 0 -> 3

Commit message: Schematic+
Parts:
- added C3: pF, symbol Device:C
- added F1: Fuse, symbol Device:Fuse
- added G10: mΩ^{-1}, symbol Device:R_US
- added L1: nH, symbol Device:L
- added R1: R_US, symbol Device:R_US
- added R9: mΩ, symbol Device:R_US
- renumbered J2 to J1, J1 to J2, R1 to R2, R2 to R3, R3 to R4, R4 to R5, R5 to R6, R6 to R7, R7 to R8
Connections:
- net AC_Pin1: now also F1.1; no longer T1.1 (AA)
- net AC_Rectified_V+: now also R1.1; no longer D5.1 (K)
- new net: L1.1, R9.2
- new net: C3.1, G10.2, L1.2
- new net: D5.1 (K), R1.2
- new net: F1.2, T1.1 (AA)
- new net GNDD: C3.2, G10.1
- no-connect marks 3 -> 4
Other:
- note added: "P_{loss} = (V_{in} - V_{out})*I P = (20V_{DC} - 5V_{DC})*0.2A = 3W"
- note added: "Protection"
- note added: "V_{DC, peak} = V_{rms}*sqrt(2) - 2V_{D} V_{D} = 0.7V_{DC} 21.2V_{pk} - 1.4V = 19.8V_{DC, pk}"
- note added: "V_{out} = V_{Z} = 15V V_{R} = 19.8V_{DC, pk} - 15V_{Z} V_{R} = 4.8V_{DC} I_{R} = (V_{DC, pk} - V_{Z}) / R_{S} I_{R} = I_{load} + I_{Z} I_{Z} = (V_{DC, pk} - V_{Z}) / R_{S} - I_{load} At I_{load} = 100mA: I_{Z, min} = 10mA I_{R} = 100mA + 10mA = 110mA R_{S} = (19.8V_{DC, pk} - 15V_{Z}) / 0.110A = 43.6Ω P_{R} = V_{R}*I_{R} P_{R} = 4.8V - 0.110A = 0.53W 1 watt resistor..."
- note added: "V_{primary}/V_{secondary} = N_{primary}/N_{secondary} V_{p} = 120Vrms, V_{s} = 15Vrms 120/15 = 8:1 turns I_{primary}/I_{secondary} = N_{secondary}/N_{primary} V_{p}I_{p} = V_{s}I_{s} VA = V_{secondary, rms}I_{secondary,rms} approx. 20VA V_{pk} = V_{rms}*sqrt(2) 15V_{rms}*sqrt(2) = 21.2V_{pk}"
- note added: "V_{rms} = VAC = V_{AC}"
- note added: "V_{rms} = V_{pk}/sqrt(2) 120V_{rms} = 169.7V_{pk}/1.414 V_{time} = A*cos(2πƒt + Θ) ƒ = 60Hz T = 16.~{66}ms λ = v/ƒ %50*c/60Hz = 2.5km"
- note added: "ΔV = I_{load}/ƒ_{ripple}*C ƒ_{ripple} = 120 Hz At I = 100mA and C = 470uF: ΔV = 0.1A/120Hz*0.00047F ΔV = 1.77V So, 19V_{DC} ±0.8V_{DC ripple}"
- company: (none) -> Lamar University | IEEE
- title: (none) -> IEEE Workshop PCB | Electronics | Hardware | Design Engineering
- moved on the sheet: C1, C2, D1, D2, D3, D4, D5, D6, J1, J2, Q1, R2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

Commit message: Testing commit
Other:
- note removed: "V_{rms} = VAC = V_{AC}"
- moved on the sheet: C1, C2, C3, D1, D2, D3, D4, D5, D6, F1, G10, J1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

Commit message: Work Anas
Parts:
- removed C2: C, symbol Device:C
- removed C3: pF, symbol Device:C
- removed G10: mΩ^{-1}, symbol Device:R_US
- removed J1: Screw_Terminal_01x03, symbol Connector:Screw_Terminal_01x03
- removed L1: nH, symbol Device:L
- removed Q1: RS9N50D, Package_TO_SOT_SMD:TO-252-2, symbol Transistor_FET:RS9N50D
- removed R2, R3, R6, R7: R_US, symbol Device:R_US
- removed R4, R5: R, symbol Device:R_Small_US
- removed R9: mΩ, symbol Device:R_US
- removed unit 3 of U1
- removed unit 1 of U1
- added J3: Screw_Terminal_01x02, Connector_Molex:Molex_Mini-Fit_Jr_5569-06A1_2x03_P4.20mm_Horizontal, symbol Connector:Screw_Terminal_01x02
- added Q1: 2SD600, Package_TO_SOT_THT:TO-126-3_Vertical, symbol Transistor_BJT:2SD600
- added R10: R_US, Resistor_THT:R_Axial_DIN0204_L3.6mm_D1.6mm_P7.62mm_Horizontal, symbol Device:R_US
- added RV1: R_Potentiometer_US, symbol Device:R_Potentiometer_US
- added U2: TLV172IDCK, Package_TO_SOT_SMD:SOT-353_SC-70-5, symbol Amplifier_Operational:TLV172IDCK
- C1: footprint (none) -> Capacitor_THT:CP_Radial_D10.0mm_P3.50mm
- D1, D2, D3, D4, D5: footprint (none) -> Diode_THT:D_DO-35_SOD27_P7.62mm_Horizontal
- D6: footprint (none) -> LED_THT:LED_D5.0mm
- J2: footprint (none) -> Connector_Molex:Molex_Mini-Fit_Jr_5569-06A1_2x03_P4.20mm_Horizontal
- R1, R8: footprint (none) -> Resistor_THT:R_Axial_DIN0204_L3.6mm_D1.6mm_P7.62mm_Horizontal
Connections:
- net VirtualGND is gone; now on net AC_Rectified_V-: J2.2 (Pin_2), R8.2
- net AC_Pin1: now also J3.2 (Pin_2)
- net AC_Pin2: now also J3.1 (Pin_1)
- net AC_Rectified_V+: now also Q1.2 (C), U2.5 (V+)
- net AC_Rectified_V-: now also RV1.1, U2.2 (V-)
- net at D6.2 (A), J2.1 (Pin_1): now also Q1.1 (E), R10.1
- net at D5.1 (K), R1.2: now also U2.1 (+)
- new net: R10.2, RV1.3
- new net: RV1.2, U2.3 (-)
- new net: Q1.3 (B), U2.4
- no-connect marks 4 -> 3
Other:
- note removed: "P_{loss} = (V_{in} - V_{out})*I P = (20V_{DC} - 5V_{DC})*0.2A = 3W"
- moved on the sheet: D6, J2, R8

Commit message: Net Labels
Parts:
- D5: value D_Zener -> 1V
- D6: value LED -> Red
- R1: value R_US -> 10k
- R10: value R_US -> 680
- R8: value R_US -> 220
- RV1: value R_Potentiometer_US -> 1K
Connections:
- net Vout: now reaches D6.2 (A), J2.1 (Pin_1), Q1.1 (E), R10.1
- net VRef: now reaches D5.1 (K), R1.2, U2.1 (+)
- net Vfdbck: now reaches RV1.2, U2.3 (-)
Other:
- moved on the sheet: C1, D6, J2, Q1, R8, U2

Commit message: 9/2 - Layout and Schematic
Parts:
- removed J2, J3: Screw_Terminal_01x02, Connector_Molex:Molex_Mini-Fit_Jr_5569-06A1_2x03_P4.20mm_Horizontal, symbol Connector:Screw_Terminal_01x02
- removed T1: Transformer_1P_1S, symbol Device:Transformer_1P_1S
- removed U1: Opamp_Dual, symbol Device:Opamp_Dual
- added F2: 1A, Fuse:Fuseholder_Clip-5x20mm_Keystone_3517_Inline_P23.11x6.76mm_D1.70mm_Horizontal, symbol Device:Fuse
- added J1, J2: Screw_Terminal_01x03, TerminalBlock_Phoenix:TerminalBlock_Phoenix_MKDS-1,5-3_1x03_P5.00mm_Horizontal, symbol Connector:Screw_Terminal_01x03
- added R1, R2, R3: 0, Resistor_THT:R_Axial_DIN0309_L9.0mm_D3.2mm_P12.70mm_Horizontal, symbol Device:R_US
- added TR1: VPP12-200, Transformer_THT:XFMR_VPP12-200, symbol Transformer:TRANSF6
- C1: footprint Capacitor_THT:CP_Radial_D10.0mm_P3.50mm -> Capacitor_THT:CP_Radial_D8.0mm_P3.50mm
- F1: value Fuse -> 100mA; footprint (none) -> Fuse:Fuseholder_Clip-5x20mm_Keystone_3517_Inline_P23.11x6.76mm_D1.70mm_Horizontal
- Q1: footprint Package_TO_SOT_THT:TO-126-3_Vertical -> Package_TO_SOT_THT:TO-92_Inline_Wide
- R4: renamed from R1; footprint Resistor_THT:R_Axial_DIN0204_L3.6mm_D1.6mm_P7.62mm_Horizontal -> Resistor_THT:R_Axial_DIN0309_L9.0mm_D3.2mm_P12.70mm_Horizontal
- R5: renamed from R10; footprint Resistor_THT:R_Axial_DIN0204_L3.6mm_D1.6mm_P7.62mm_Horizontal -> Resistor_THT:R_Axial_DIN0309_L9.0mm_D3.2mm_P12.70mm_Horizontal
- R6: renamed from R8; footprint Resistor_THT:R_Axial_DIN0204_L3.6mm_D1.6mm_P7.62mm_Horizontal -> Resistor_THT:R_Axial_DIN0309_L9.0mm_D3.2mm_P12.70mm_Horizontal
- RV1: value 1K -> 10k; footprint (none) -> Potentiometer_THT:Potentiometer_Runtron_RM-063_Horizontal
- U1: renamed from U2; footprint Package_TO_SOT_SMD:SOT-353_SC-70-5 -> Package_DIP:DIP-8_W7.62mm_LongPads
Connections:
- net T2 is gone; now on net GND2: D2.1 (K), D4.2 (A)
- net AC_Pin1: now also J1.3 (Pin_3)
- net T1: now also F2.2, R2.1
- net Vout: now also J2.1 (Pin_1)
- net at F1.2: now also TR1.1, TR1.3
- net AC_Rectified_V- renamed GND2
- net GND2: now also J2.2 (Pin_2), R1.2, TR1.5
- new net C1+: F2.1, TR1.8
- new net C1-: R1.1, R3.2, TR1.7
- new net C2+: R2.2, R3.1, TR1.6
- new net GND1: J1.1 (Pin_1), J1.2 (Pin_2), J2.3 (Pin_3), TR1.2, TR1.4
- no-connect marks 3 -> 0
Other:
- note removed: "Protection"
- moved on the sheet: C1, D1, D2, D3, D4, D5, D6, F1, Q1, R4, R5, R6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

Commit message: Almost Done
Parts:
- D1, D2, D3, D4: value D_45deg -> 1N4007GP-AQ
- J1: value Screw_Terminal_01x03 -> TB002-500-02BE
- Q1: value 2SD600 -> BC63916-D27Z
- R1, R2: now fitted
- U1: value TLV172IDCK -> LM358P
Connections:
- net AC_Rectified_V+: now also U1.8 (V+); no longer U1.5 (V+)
- net GND1: now also C1.2, D1.2 (A), D2.1 (K), D2.2 (A), D4.2 (A), D5.2 (A), J2.2 (Pin_2), R1.2, R6.2, RV1.1, TR1.5, U1.4 (V-)
- net VRef: now also U1.3 (+); no longer U1.1 (+)
- net Vfdbck: now also U1.2 (-); no longer U1.3 (-)
- net at Q1.3 (B): now also U1.1; no longer U1.4
- net AC_Pin1 renamed +
- net C1+ renamed S1+
- net C1- renamed S1-
- net C2+ renamed S2+
- removed net GND2: C1.2, D1.2 (A), D2.1 (K), D2.2 (A), D4.2 (A), D5.2 (A), J2.2 (Pin_2), R1.2, R6.2, RV1.1, TR1.5, U1.2 (V-)
- net T1: no longer names the net of D1.1 (K), D3.2 (A), F2.2, R2.1
Other:
- company: Lamar University | IEEE -> Lamar University
- title: IEEE Workshop PCB | Electronics | Hardware | Design Engineering -> IEEE PCB Design Series 2026
- moved on the sheet: C1, D1, D2, D3, D4, D5, D6, F1, F2, J1, J2, Q1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

Commit message: Update
Parts:
- removed D5: 1V, Diode_THT:D_DO-35_SOD27_P7.62mm_Horizontal, symbol Device:D_Zener
- removed R1, R2, R3: 0, Resistor_THT:R_Axial_DIN0309_L9.0mm_D3.2mm_P12.70mm_Horizontal, symbol Device:R_US
- added R5: 10k, Resistor_THT:R_Axial_DIN0309_L9.0mm_D3.2mm_P12.70mm_Horizontal, symbol Device:R_US
- F1: value 100mA -> 1A
- renumbered D6 to D5, R5 to R6, R6 to R7
Connections:
- net S2+ is gone; now on net S1-: TR1.6
- net VRef: now also R5.1
- removed net GND1: C1.2, D1.2 (A), D2.1 (K), D2.2 (A), D4.2 (A), J1.1 (Pin_1), J1.2 (Pin_2), J2.2 (Pin_2), J2.3 (Pin_3), R7.2, RV1.1, TR1.2, TR1.4, TR1.5, U1.4 (V-)
- new net -: J1.2 (Pin_2), TR1.2, TR1.4
- new net GND2: C1.2, D1.2 (A), D2.2 (A), J2.2 (Pin_2), R5.2, R7.2, RV1.1, U1.4 (V-)
- new net GNDPWR: J1.1 (Pin_1), J2.3 (Pin_3)
- new net S2-: D2.1 (K), D4.2 (A), TR1.5
Other:
- note removed: "V_{out} = V_{Z} = 15V V_{R} = 19.8V_{DC, pk} - 15V_{Z} V_{R} = 4.8V_{DC} I_{R} = (V_{DC, pk} - V_{Z}) / R_{S} I_{R} = I_{load} + I_{Z} I_{Z} = (V_{DC, pk} - V_{Z}) / R_{S} - I_{load} At I_{load} = 100mA: I_{Z, min} = 10mA I_{R} = 100mA + 10mA = 110mA R_{S} = (19.8V_{DC, pk} - 15V_{Z}) / 0.110A = 43.6Ω P_{R} = V_{R}*I_{R} P_{R} = 4.8V - 0.110A = 0.53W 1 watt resistor..."
- moved on the sheet: C1, D1, D2, D3, D4, D5, F1, F2, J2, Q1, R4, R6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
