File: IEEE_Wrkshp_08192026.kicad_sch (KiCad schematic)
At the start: 18 parts, among them J1 TB002-500-02BE, J2 Screw_Terminal_01x03, Q1 BC63916-D27Z, U1 LM358P

Commit message: update 2
Parts:
- added TP2, TP3: TestPoint_2Pole, TestPoint:TestPoint_2Pads_Pitch2.54mm_Drill0.8mm, symbol Connector:TestPoint_2Pole
Connections:
- net AC_Rectified_V+: now also TP3.1
- net GND2: now also TP2.2, TP3.2
- net Vout: now also TP2.1

Commit message: Update
Parts:
- removed F2: 1A, Fuse:Fuseholder_Clip-5x20mm_Keystone_3517_Inline_P23.11x6.76mm_D1.70mm_Horizontal, symbol Device:Fuse
- removed R5: 10k, Resistor_THT:R_Axial_DIN0309_L9.0mm_D3.2mm_P12.70mm_Horizontal, symbol Device:R_US
- added RV2: 10k, Potentiometer_THT:Potentiometer_Runtron_RM-063_Horizontal, symbol Device:R_Potentiometer_US
Connections:
- net GND2: now also RV2.3
- net S1+: now also D1.1 (K), D3.2 (A)
- net VRef: now also RV2.2; no longer R4.2
- new net: R4.2, RV2.1
Other:
- moved on the sheet: C1, R4, TP3

Commit message: up
Parts:
- J2: value Screw_Terminal_01x03 -> TB002-500-02BE
Changed lines of the file:
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@@
 	(text "V_{rms} = V_{pk}/sqrt(2)\n120V_{rms} = 169.7V_{pk}/1.414\n\nV_{time} = A*cos(2πƒt + Θ)\n\nƒ = 60Hz\nT = 16.~{66}ms\n\nλ = v/ƒ\n%50*c/60Hz = 2.5km"
 		(exclude_from_sim no)
-		(at 33.274 114.554 0)
+		(at 50.292 239.014 0)
 		(effects
 			(font
@@
 	(text "V_{DC, peak} = V_{rms}*sqrt(2) - 2V_{D}\nV_{D} = 0.7V_{DC}\n21.2V_{pk} - 1.4V = 19.8V_{DC, pk}"
 		(exclude_from_sim no)
-		(at 92.964 122.428 0)
+		(at 109.982 246.888 0)
 		(effects
 			(font
@@
 	(text "ΔV = I_{load}/ƒ_{ripple}*C\nƒ_{ripple} = 120 Hz\n\nAt I = 100mA and C = 470uF:\nΔV = 0.1A/120Hz*0.00047F\nΔV = 1.77V\n\nSo, 19V_{DC} ±0.8V_{DC ripple}"
 		(exclude_from_sim no)
-		(at 116.078 120.65 0)
+		(at 133.096 245.11 0)
 		(effects
 			(font
@@
 	(text "V_{primary}/V_{secondary} = N_{primary}/N_{secondary}\nV_{p} = 120Vrms, V_{s} = 15Vrms\n120/15 = 8:1 turns\n\nI_{primary}/I_{secondary} = N_{secondary}/N_{primary}\nV_{p}I_{p} = V_{s}I_{s}\nVA = V_{secondary, rms}I_{secondary,rms}\napprox. 20VA\n\nV_{pk} = V_{rms}*sqrt(2)\n15V_{rms}*sqrt(2) = 21.2V_{pk}"
 		(exclude_from_sim no)
-		(at 53.34 117.856 0)
+		(at 70.358 242.316 0)
 		(effects
 			(font
@@
 			)
 		)
-		(property "Value" "Screw_Terminal_01x03"
+		(property "Value" "TB002-500-02BE"
 			(at 227.33 93.98 0)
 			(show_name no)
